File: ir_board.sch (EAGLE design)
At the start: 13 parts

Commit message: Added debounce caps
Parts:
- added C1, C2: (no value), rcl:C-EUC0805K
Connections:
- net GND: now also C1.1, C2.1
- net VCC: now also C1.2, C2.2
Changed lines of the file:
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@@
 <part name="GND6" library="supply1" deviceset="GND" device=""/>
 <part name="R6" library="rcl" deviceset="R-US_" device="R0805" value="0ohm"/>
+<part name="C1" library="rcl" deviceset="C-EU" device="C0805K"/>
+<part name="C2" library="rcl" deviceset="C-EU" device="C0805K"/>
 </parts>
 <sheets>
@@
 <instance part="GND6" gate="1" x="53.34" y="5.08"/>
 <instance part="R6" gate="G$1" x="81.28" y="101.6"/>
+<instance part="C1" gate="G$1" x="88.9" y="33.02"/>
+<instance part="C2" gate="G$1" x="99.06" y="33.02"/>
 </instances>
 <busses>
@@
 <junction x="60.96" y="35.56"/>
 <junction x="76.2" y="35.56"/>
+<pinref part="C1" gate="G$1" pin="1"/>
+<wire x1="88.9" y1="35.56" x2="76.2" y2="35.56" width="0.1524" layer="91"/>
+<pinref part="C2" gate="G$1" pin="1"/>
+<wire x1="76.2" y1="35.56" x2="88.9" y2="35.56" width="0.1524" layer="91"/>
+<junction x="88.9" y="35.56"/>
+<wire x1="88.9" y1="35.56" x2="99.06" y2="35.56" width="0.1524" layer="91"/>
+<junction x="99.06" y="35.56"/>
 </segment>
 <segment>
@@
 </segment>
 <segment>
-<wire x1="66.04" y1="30.48" x2="60.96" y2="30.48" width="0.1524" layer="91"/>
+<wire x1="66.04" y1="30.48" x2="63.5" y2="30.48" width="0.1524" layer="91"/>
 <pinref part="U$3" gate="G$1" pin="VCC"/>
 <junction x="60.96" y="30.48"/>
 <label x="66.04" y="30.48" size="1.778" layer="95"/>
-</segment>
-<segment>
+<wire x1="63.5" y1="30.48" x2="60.96" y2="30.48" width="0.1524" layer="91"/>
+<wire x1="63.5" y1="30.48" x2="63.5" y2="27.94" width="0.1524" layer="91"/>
+<pinref part="C1" gate="G$1" pin="2"/>
+<wire x1="63.5" y1="27.94" x2="88.9" y2="27.94" width="0.1524" layer="91"/>
+<pinref part="C2" gate="G$1" pin="2"/>
+<wire x1="88.9" y1="27.94" x2="99.06" y2="27.94" width="0.1524" layer="91"/>
+<junction x="88.9" y="27.94"/>
+<junction x="99.06" y="27.94"/>
+</segment>
+<segment>
